Commit message: Change joints name of unitree_description

File: quad_example/unitree_description/urdf/common/leg.xacro (robot description, xacro)
@@ -3,5 +3,5 @@
     <xacro:include filename="$(find unitree_description)/urdf/common/transmission.xacro"/>
     <xacro:macro name="leg" params="prefix mirror mirror_dae front_hind front_hind_dae *origin">
-        <joint name="${prefix}_hip_joint" type="revolute">
+        <joint name="${prefix}_HAA" type="revolute">
             <xacro:insert_block name="origin"/>
             <parent link="base_link"/>
@@ -52,5 +52,5 @@
             </inertial>
         </link>
-        <joint name="${prefix}_thigh_joint" type="revolute">
+        <joint name="${prefix}_HFE" type="revolute">
             <origin rpy="0 0 0" xyz="0 ${thigh_offset*mirror} 0"/>
             <parent link="${prefix}_hip"/>
@@ -97,5 +97,5 @@
             </inertial>
         </link>
-        <joint name="${prefix}_calf_joint" type="revolute">
+        <joint name="${prefix}_KFE" type="revolute">
             <origin rpy="0 0 0" xyz="0 0 ${-thigh_length}"/>
             <parent link="${prefix}_thigh"/>
@@ -131,7 +131,7 @@
             <origin rpy="0 0 0" xyz="0 0 ${-(calf_length)}"/>
             <parent link="${prefix}_calf"/>
-            <child link="${prefix}_foot"/>
+            <child link="${prefix}_FOOT"/>
         </joint>
-        <link name="${prefix}_foot">
+        <link name="${prefix}_FOOT">
             <visual>
                 <origin rpy="0 0 0" xyz="0 0 0"/>

File: quad_example/unitree_description/urdf/robot.xacro (robot description, xacro)
@@ -38,14 +38,14 @@
     </link>
     <xacro:IMU connected_to="base_link" imu_name="unitree_imu" xyz="0. 0. 0." rpy="0. 0. 0."/>
-    <xacro:leg prefix="FR" mirror="-1" mirror_dae="False" front_hind="1" front_hind_dae="True">
+    <xacro:leg prefix="RF" mirror="-1" mirror_dae="False" front_hind="1" front_hind_dae="True">
         <origin rpy="0 0 0" xyz="${leg_offset_x} ${-leg_offset_y} 0"/>
     </xacro:leg>
-    <xacro:leg prefix="FL" mirror="1" mirror_dae="True" front_hind="1" front_hind_dae="True">
+    <xacro:leg prefix="LF" mirror="1" mirror_dae="True" front_hind="1" front_hind_dae="True">
         <origin rpy="0 0 0" xyz="${leg_offset_x} ${leg_offset_y} 0"/>
     </xacro:leg>
-    <xacro:leg prefix="RR" mirror="-1" mirror_dae="False" front_hind="-1" front_hind_dae="False">
+    <xacro:leg prefix="RH" mirror="-1" mirror_dae="False" front_hind="-1" front_hind_dae="False">
         <origin rpy="0 0 0" xyz="${-leg_offset_x} ${-leg_offset_y} 0"/>
     </xacro:leg>
-    <xacro:leg prefix="RL" mirror="1" mirror_dae="True" front_hind="-1" front_hind_dae="False">
+    <xacro:leg prefix="LH" mirror="1" mirror_dae="True" front_hind="-1" front_hind_dae="False">
         <origin rpy="0 0 0" xyz="${-leg_offset_x} ${leg_offset_y} 0"/>
     </xacro:leg>
