Commit message: Replace "base_link" with "base" in all URDF

File: quad_example/unitree_description/urdf/a1.urdf (robot description, URDF)
Before this commit: robot robot, 18 links, 17 joints
Links:
- removed link base_link
- added link base, mass 6.0; collision box size=0.267 0.194 0.114; visual mesh filename=package://unitree_description/meshes/a1/trunk.dae scale=1 1 1
Joints:
- joint LF_HAA: parent base_link -> base
- joint LH_HAA: parent base_link -> base
- joint RF_HAA: parent base_link -> base
- joint RH_HAA: parent base_link -> base
- joint unitree_imu_joint: parent base_link -> base

File: quad_example/unitree_description/urdf/common/gazebo.xacro (robot description, xacro)
@@ -13,5 +13,5 @@
             <alwaysOn>true</alwaysOn>
             <updateRate>1000.0</updateRate>
-            <bodyName>base_link</bodyName>
+            <bodyName>base</bodyName>
             <topicName>ground_truth/state</topicName>
             <gaussianNoise>0</gaussianNoise>

File: quad_example/unitree_description/urdf/common/leg.xacro (robot description, xacro)
@@ -5,5 +5,5 @@
         <joint name="${prefix}_HAA" type="revolute">
             <xacro:insert_block name="origin"/>
-            <parent link="base_link"/>
+            <parent link="base"/>
             <child link="${prefix}_hip"/>
             <axis xyz="1 0 0"/>

File: quad_example/unitree_description/urdf/robot.xacro (robot description, xacro)
@@ -7,13 +7,5 @@
     <xacro:include filename="$(find unitree_description)/urdf/common/imu.xacro"/>
     <xacro:include filename="$(find unitree_description)/urdf/$(arg robot_type)/const.xacro"/>
-    <xacro:if value="$(arg hung_up)">
-        <link name="world"/>
-        <joint name="base_static_joint" type="fixed">
-            <origin rpy="0 0 0" xyz="0 0 0"/>
-            <parent link="world"/>
-            <child link="base_link"/>
-        </joint>
-    </xacro:if>
-    <link name="base_link">
+    <link name="base">
         <visual>
             <origin rpy="0 0 0" xyz="0 0 0"/>
@@ -37,5 +29,5 @@
         </inertial>
     </link>
-    <xacro:IMU connected_to="base_link" imu_name="unitree_imu" xyz="0. 0. 0." rpy="0. 0. 0."/>
+    <xacro:IMU connected_to="base" imu_name="unitree_imu" xyz="0. 0. 0." rpy="0. 0. 0."/>
     <xacro:leg prefix="RF" mirror="-1" mirror_dae="False" front_hind="1" front_hind_dae="True">
         <origin rpy="0 0 0" xyz="${leg_offset_x} ${-leg_offset_y} 0"/>
