Commit message: Rename unitree_description to legged_unitree_description

File: legged_examples/legged_unitree/legged_unitree_description/urdf/a1.urdf (robot description, URDF)
Before this commit: robot robot, 18 links, 17 joints
Links:
- link LF_calf: geometry collision box size=0.2 0.016 0.016; visual mesh filename=package://legged_unitree_description/meshes/a1/calf.dae scale=1 1 1
- link LF_hip: geometry collision cylinder length=0.04 radius=0.046; visual mesh filename=package://legged_unitree_description/meshes/a1/hip.dae scale=1 1 1
- link LF_thigh: geometry collision box size=0.2 0.0245 0.034; collision cylinder length=0.032 radius=0.041
- link LH_calf: geometry collision box size=0.2 0.016 0.016; visual mesh filename=package://legged_unitree_description/meshes/a1/calf.dae scale=1 1 1
- link LH_hip: geometry collision cylinder length=0.04 radius=0.046; visual mesh filename=package://legged_unitree_description/meshes/a1/hip.dae scale=1 1 1
- link LH_thigh: geometry collision box size=0.2 0.0245 0.034; collision cylinder length=0.032 radius=0.041
- link RF_calf: geometry collision box size=0.2 0.016 0.016; visual mesh filename=package://legged_unitree_description/meshes/a1/calf.dae scale=1 1 1
- link RF_hip: geometry collision cylinder length=0.04 radius=0.046; visual mesh filename=package://legged_unitree_description/meshes/a1/hip.dae scale=1 1 1
- link RF_thigh: geometry collision box size=0.2 0.0245 0.034; collision cylinder length=0.032 radius=0.041
- link RH_calf: geometry collision box size=0.2 0.016 0.016; visual mesh filename=package://legged_unitree_description/meshes/a1/calf.dae scale=1 1 1
- link RH_hip: geometry collision cylinder length=0.04 radius=0.046; visual mesh filename=package://legged_unitree_description/meshes/a1/hip.dae scale=1 1 1
- link RH_thigh: geometry collision box size=0.2 0.0245 0.034; collision cylinder length=0.032 radius=0.041
- link base: geometry collision box size=0.267 0.194 0.114; visual mesh filename=package://legged_unitree_description/meshes/a1/trunk.dae scale=1 1 1

File: legged_examples/legged_unitree/legged_unitree_description/urdf/common/leg.xacro (robot description, xacro)
@@ -1,5 +1,5 @@
 <?xml version="1.0"?>
 <robot xmlns:xacro="http://www.ros.org/wiki/xacro">
-    <xacro:include filename="$(find unitree_description)/urdf/common/transmission.xacro"/>
+    <xacro:include filename="$(find legged_unitree_description)/urdf/common/transmission.xacro"/>
     <xacro:macro name="leg" params="prefix mirror mirror_dae front_hind front_hind_dae *origin">
         <joint name="${prefix}_HAA" type="revolute">
@@ -33,5 +33,6 @@
                 </xacro:if>
                 <geometry>
-                    <mesh filename="package://unitree_description/meshes/$(arg robot_type)/hip.dae" scale="1 1 1"/>
+                    <mesh filename="package://legged_unitree_description/meshes/$(arg robot_type)/hip.dae"
+                          scale="1 1 1"/>
                 </geometry>
                 <material name="orange"/>
@@ -66,9 +67,9 @@
                 <geometry>
                     <xacro:if value="${mirror_dae == True}">
-                        <mesh filename="package://unitree_description/meshes/$(arg robot_type)/thigh.dae"
+                        <mesh filename="package://legged_unitree_description/meshes/$(arg robot_type)/thigh.dae"
                               scale="1 1 1"/>
                     </xacro:if>
                     <xacro:if value="${mirror_dae == False}">
-                        <mesh filename="package://unitree_description/meshes/$(arg robot_type)/thigh_mirror.dae"
+                        <mesh filename="package://legged_unitree_description/meshes/$(arg robot_type)/thigh_mirror.dae"
                               scale="1 1 1"/>
                     </xacro:if>
@@ -109,5 +110,6 @@
                 <origin rpy="0 0 0" xyz="0 0 0"/>
                 <geometry>
-                    <mesh filename="package://unitree_description/meshes/$(arg robot_type)/calf.dae" scale="1 1 1"/>
+                    <mesh filename="package://legged_unitree_description/meshes/$(arg robot_type)/calf.dae"
+                          scale="1 1 1"/>
                 </geometry>
                 <material name="orange"/>

File: legged_examples/legged_unitree/legged_unitree_description/urdf/robot.xacro (robot description, xacro)
@@ -2,14 +2,14 @@
 <robot xmlns:xacro="http://www.ros.org/wiki/xacro" name="robot">
     <xacro:arg name="robot_type" default="a1"/>
-    <xacro:include filename="$(find unitree_description)/urdf/common/materials.xacro"/>
-    <xacro:include filename="$(find unitree_description)/urdf/common/leg.xacro"/>
-    <xacro:include filename="$(find unitree_description)/urdf/common/gazebo.xacro"/>
-    <xacro:include filename="$(find unitree_description)/urdf/common/imu.xacro"/>
-    <xacro:include filename="$(find unitree_description)/urdf/$(arg robot_type)/const.xacro"/>
+    <xacro:include filename="$(find legged_unitree_description)/urdf/common/materials.xacro"/>
+    <xacro:include filename="$(find legged_unitree_description)/urdf/common/leg.xacro"/>
+    <xacro:include filename="$(find legged_unitree_description)/urdf/common/gazebo.xacro"/>
+    <xacro:include filename="$(find legged_unitree_description)/urdf/common/imu.xacro"/>
+    <xacro:include filename="$(find legged_unitree_description)/urdf/$(arg robot_type)/const.xacro"/>
     <link name="base">
         <visual>
             <origin rpy="0 0 0" xyz="0 0 0"/>
             <geometry>
-                <mesh filename="package://unitree_description/meshes/$(arg robot_type)/trunk.dae" scale="1 1 1"/>
+                <mesh filename="package://legged_unitree_description/meshes/$(arg robot_type)/trunk.dae" scale="1 1 1"/>
             </geometry>
         </visual>

Commit message: More precise collision model of a1

File: legged_examples/legged_unitree/legged_unitree_description/urdf/a1.urdf (robot description, URDF)
Before this commit: robot robot, 18 links, 17 joints
Links:
- link LF_thigh: geometry collision box size=0.2 0.03 0.034; collision cylinder length=0.04 radius=0.041
- link LH_thigh: geometry collision box size=0.2 0.03 0.034; collision cylinder length=0.04 radius=0.041
- link RF_thigh: geometry collision box size=0.2 0.03 0.034; collision cylinder length=0.04 radius=0.041
- link RH_thigh: geometry collision box size=0.2 0.03 0.034; collision cylinder length=0.04 radius=0.041

File: legged_examples/legged_unitree/legged_unitree_description/urdf/a1/const.xacro (robot description, xacro)
@@ -10,6 +10,8 @@
     <xacro:property name="hip_length" value="0.04"/>
     <xacro:property name="thigh_shoulder_radius" value="0.041"/>
-    <xacro:property name="thigh_shoulder_length" value="0.032"/>
-    <xacro:property name="thigh_width" value="0.0245"/>
+    <xacro:property name="thigh_shoulder_length" value="0.04"/>
+    <xacro:property name="thigh_shoulder_y_offset" value="-0.008"/>
+    <xacro:property name="thigh_x_offset" value="-0.015"/>
+    <xacro:property name="thigh_width" value="0.03"/>
     <xacro:property name="thigh_height" value="0.034"/>
     <xacro:property name="calf_width" value="0.016"/>

File: legged_examples/legged_unitree/legged_unitree_description/urdf/common/leg.xacro (robot description, xacro)
@@ -78,5 +78,5 @@
             </visual>
             <collision>
-                <origin rpy="0 ${pi/2.0} 0" xyz="0 0 ${-thigh_length/2.0}"/>
+                <origin rpy="0 ${pi/2.0+0.1} 0" xyz="${thigh_x_offset} 0 ${-thigh_length/2.0}"/>
                 <geometry>
                     <box size="${thigh_length} ${thigh_width} ${thigh_height}"/>
@@ -84,5 +84,5 @@
             </collision>
             <collision>
-                <origin rpy="${pi/2.0} 0 0" xyz="0 0 0"/>
+                <origin rpy="${pi/2.0} 0 0" xyz="0 ${mirror*thigh_shoulder_y_offset} 0"/>
                 <geometry>
                     <cylinder length="${thigh_shoulder_length}" radius="${thigh_shoulder_radius}"/>
