Commit message: Simplify urdf

File: legged_examples/legged_unitree/legged_unitree_description/urdf/common/leg.xacro (robot description, xacro)
@@ -160,4 +160,30 @@
             <disableFixedJointLumping>true</disableFixedJointLumping>
         </gazebo>
+        <gazebo reference="${prefix}_hip">
+            <mu1>0.2</mu1>
+            <mu2>0.2</mu2>
+            <material>Gazebo/DarkGrey</material>
+        </gazebo>
+        <gazebo reference="${prefix}_thigh">
+            <mu1>0.2</mu1>
+            <mu2>0.2</mu2>
+            <self_collide>0</self_collide>
+            <material>Gazebo/DarkGrey</material>
+            <kp value="1000000.0"/>
+            <kd value="100.0"/>
+        </gazebo>
+        <gazebo reference="${prefix}_calf">
+            <mu1>0.6</mu1>
+            <mu2>0.6</mu2>
+            <self_collide>1</self_collide>
+        </gazebo>
+        <gazebo reference="${prefix}_FOOT">
+            <mu1>0.6</mu1>
+            <mu2>0.6</mu2>
+            <self_collide>1</self_collide>
+            <material>Gazebo/DarkGrey</material>
+            <kp value="1000000.0"/>
+            <kd value="100.0"/>
+        </gazebo>
         <xacro:leg_transmission name="${prefix}"/>
     </xacro:macro>

Commit message: Use more precise leg foot contact in leg urdf

File: legged_examples/legged_unitree/legged_unitree_description/urdf/common/leg.xacro (robot description, xacro)
@@ -123,13 +123,13 @@
             <inertial>
                 <origin rpy="0 0 0" xyz="${calf_com_x} ${calf_com_y} ${calf_com_z}"/>
-                <mass value="${calf_mass}"/>
+                <mass value="${calf_mass/2}"/>
                 <inertia
-                        ixx="${calf_ixx}" ixy="${calf_ixy}" ixz="${calf_ixz}"
-                        iyy="${calf_iyy}" iyz="${calf_iyz}"
-                        izz="${calf_izz}"/>
+                        ixx="${calf_ixx/2}" ixy="${calf_ixy/2}" ixz="${calf_ixz/2}"
+                        iyy="${calf_iyy/2}" iyz="${calf_iyz/2}"
+                        izz="${calf_izz/2}"/>
             </inertial>
         </link>
         <joint name="${prefix}_foot_fixed" type="fixed">
-            <origin rpy="0 0 0" xyz="0 0 ${-(calf_length)}"/>
+            <origin rpy="0 0 0" xyz="${-0.707*foot_radius} 0 ${-calf_length-0.707*foot_radius}"/>
             <parent link="${prefix}_calf"/>
             <child link="${prefix}_FOOT"/>
@@ -137,5 +137,5 @@
         <link name="${prefix}_FOOT">
             <visual>
-                <origin rpy="0 0 0" xyz="0 0 0"/>
+                <origin rpy="0 0 0" xyz="${0.707*foot_radius} 0 ${0.707*foot_radius}"/>
                 <geometry>
                     <sphere radius="${foot_radius-0.01}"/>
@@ -144,5 +144,5 @@
             </visual>
             <collision>
-                <origin rpy="0 0 0" xyz="0 0 0"/>
+                <origin rpy="0 0 0" xyz="${0.707*foot_radius} 0 ${0.707*foot_radius}"/>
                 <geometry>
                     <sphere radius="${foot_radius}"/>
@@ -150,9 +150,11 @@
             </collision>
             <inertial>
-                <mass value="${foot_mass}"/>
+                <origin rpy="0 0 0"
+                        xyz="${calf_com_x+0.707*foot_radius} ${calf_com_y} ${calf_com_z+calf_length+0.707*foot_radius}"/>
+                <mass value="${calf_mass/2}"/>
                 <inertia
-                        ixx="${(2*foot_mass)/5.0*(foot_radius*foot_radius)}" ixy="0.0" ixz="0.0"
-                        iyy="${(2*foot_mass)/5.0*(foot_radius*foot_radius)}" iyz="0.0"
-                        izz="${(2*foot_mass)/5.0*(foot_radius*foot_radius)}"/>
+                        ixx="${calf_ixx/2}" ixy="${calf_ixy/2}" ixz="${calf_ixz/2}"
+                        iyy="${calf_iyy/2}" iyz="${calf_iyz/2}"
+                        izz="${calf_izz/2}"/>
             </inertial>
         </link>

Commit message: Correct collision of urdf

File: legged_examples/legged_unitree/legged_unitree_description/urdf/common/leg.xacro (robot description, xacro)
@@ -116,5 +116,5 @@
             </visual>
             <collision>
-                <origin rpy="0 ${pi/2.0} 0" xyz="0 0 ${-calf_length/2.0}"/>
+                <origin rpy="0 ${pi/2.0} 0" xyz="${calf_x_offset} 0 ${-calf_length/2.0}"/>
                 <geometry>
                     <box size="${calf_length} ${calf_width} ${calf_height}"/>

Commit message: Add go1 xarco

File: legged_examples/legged_unitree/legged_unitree_description/urdf/common/leg.xacro (robot description, xacro)
@@ -10,10 +10,10 @@
             <dynamics damping="${damping}" friction="${friction}"/>
             <xacro:if value="${(mirror_dae == True)}">
-                <limit effort="${hip_torque_max}" velocity="${hip_velocity_max}" lower="${hip_min}"
-                       upper="${hip_max}"/>
+                <limit effort="${hip_torque_max}" velocity="${hip_velocity_max}" lower="${hip_position_min}"
+                       upper="${hip_position_max}"/>
             </xacro:if>
             <xacro:if value="${(mirror_dae == False)}">
-                <limit effort="${hip_torque_max}" velocity="${hip_velocity_max}" lower="${-hip_max}"
-                       upper="${-hip_min}"/>
+                <limit effort="${hip_torque_max}" velocity="${hip_velocity_max}" lower="${-hip_position_max}"
+                       upper="${-hip_position_min}"/>
             </xacro:if>
         </joint>
@@ -59,6 +59,6 @@
             <axis xyz="0 1 0"/>
             <dynamics damping="${damping}" friction="${friction}"/>
-            <limit effort="${thigh_torque_max}" velocity="${thigh_velocity_max}" lower="${thigh_min}"
-                   upper="${thigh_max}"/>
+            <limit effort="${thigh_torque_max}" velocity="${thigh_velocity_max}" lower="${thigh_position_min}"
+                   upper="${thigh_position_max}"/>
         </joint>
         <link name="${prefix}_thigh">
@@ -104,5 +104,5 @@
             <axis xyz="0 1 0"/>
             <dynamics damping="${damping}" friction="${friction}"/>
-            <limit effort="${calf_torque_max}" velocity="${calf_velocity_max}" lower="${calf_min}" upper="${calf_max}"/>
+            <limit effort="${calf_torque_max}" velocity="${calf_velocity_max}" lower="${calf_position_min}" upper="${calf_position_max}"/>
         </joint>
         <link name="${prefix}_calf">

File: legged_examples/legged_unitree/legged_unitree_description/urdf/robot.xacro (robot description, xacro)
@@ -30,15 +30,15 @@
     </link>
     <xacro:IMU connected_to="base" imu_name="unitree_imu" xyz="0. 0. 0." rpy="0. 0. 0."/>
+    <xacro:leg prefix="LF" mirror="1" mirror_dae="True" front_hind="1" front_hind_dae="True">
+        <origin rpy="0 0 0" xyz="${leg_offset_x} ${leg_offset_y} 0"/>
+    </xacro:leg>
+    <xacro:leg prefix="LH" mirror="1" mirror_dae="True" front_hind="-1" front_hind_dae="False">
+        <origin rpy="0 0 0" xyz="${-leg_offset_x} ${leg_offset_y} 0"/>
+    </xacro:leg>
     <xacro:leg prefix="RF" mirror="-1" mirror_dae="False" front_hind="1" front_hind_dae="True">
         <origin rpy="0 0 0" xyz="${leg_offset_x} ${-leg_offset_y} 0"/>
-    </xacro:leg>
-    <xacro:leg prefix="LF" mirror="1" mirror_dae="True" front_hind="1" front_hind_dae="True">
-        <origin rpy="0 0 0" xyz="${leg_offset_x} ${leg_offset_y} 0"/>
     </xacro:leg>
     <xacro:leg prefix="RH" mirror="-1" mirror_dae="False" front_hind="-1" front_hind_dae="False">
         <origin rpy="0 0 0" xyz="${-leg_offset_x} ${-leg_offset_y} 0"/>
     </xacro:leg>
-    <xacro:leg prefix="LH" mirror="1" mirror_dae="True" front_hind="-1" front_hind_dae="False">
-        <origin rpy="0 0 0" xyz="${-leg_offset_x} ${leg_offset_y} 0"/>
-    </xacro:leg>
 </robot>

Commit message: Add some urdf support for RL

File: legged_examples/legged_unitree/legged_unitree_description/urdf/common/leg.xacro (robot description, xacro)
@@ -2,5 +2,5 @@
 <robot xmlns:xacro="http://www.ros.org/wiki/xacro">
     <xacro:include filename="$(find legged_unitree_description)/urdf/common/transmission.xacro"/>
-    <xacro:macro name="leg" params="prefix mirror mirror_dae front_hind front_hind_dae *origin">
+    <xacro:macro name="leg" params="prefix mesh_path mirror mirror_dae front_hind front_hind_dae *origin">
         <joint name="${prefix}_HAA" type="revolute">
             <xacro:insert_block name="origin"/>
@@ -33,5 +33,5 @@
                 </xacro:if>
                 <geometry>
-                    <mesh filename="package://legged_unitree_description/meshes/$(arg robot_type)/hip.dae"
+                    <mesh filename="${mesh_path}/hip.dae"
                           scale="1 1 1"/>
                 </geometry>
@@ -67,9 +67,9 @@
                 <geometry>
                     <xacro:if value="${mirror_dae == True}">
-                        <mesh filename="package://legged_unitree_description/meshes/$(arg robot_type)/thigh.dae"
+                        <mesh filename="${mesh_path}/thigh.dae"
                               scale="1 1 1"/>
                     </xacro:if>
                     <xacro:if value="${mirror_dae == False}">
-                        <mesh filename="package://legged_unitree_description/meshes/$(arg robot_type)/thigh_mirror.dae"
+                        <mesh filename="${mesh_path}/thigh_mirror.dae"
                               scale="1 1 1"/>
                     </xacro:if>
@@ -110,5 +110,5 @@
                 <origin rpy="0 0 0" xyz="0 0 0"/>
                 <geometry>
-                    <mesh filename="package://legged_unitree_description/meshes/$(arg robot_type)/calf.dae"
+                    <mesh filename="${mesh_path}/calf.dae"
                           scale="1 1 1"/>
                 </geometry>
@@ -130,5 +130,5 @@
             </inertial>
         </link>
-        <joint name="${prefix}_foot_fixed" type="fixed">
+        <joint name="${prefix}_foot_fixed" type="fixed" dont_collapse="true">
             <origin rpy="0 0 0" xyz="0 0 ${-(calf_length)}"/>
             <parent link="${prefix}_calf"/>

File: legged_examples/legged_unitree/legged_unitree_description/urdf/robot.xacro (robot description, xacro)
@@ -7,9 +7,11 @@
     <xacro:include filename="$(find legged_unitree_description)/urdf/common/imu.xacro"/>
     <xacro:include filename="$(find legged_unitree_description)/urdf/$(arg robot_type)/const.xacro"/>
+<!--    <xacro:property name="mesh_path" value="../meshes"/>-->
+    <xacro:property name="mesh_path" value="$(find legged_unitree_description)/meshes/$(arg robot_type)"/>
     <link name="base">
         <visual>
             <origin rpy="0 0 0" xyz="0 0 0"/>
             <geometry>
-                <mesh filename="package://legged_unitree_description/meshes/$(arg robot_type)/trunk.dae" scale="1 1 1"/>
+                <mesh filename="${mesh_path}/trunk.dae" scale="1 1 1"/>
             </geometry>
         </visual>
@@ -30,14 +32,14 @@
     </link>
     <xacro:IMU connected_to="base" imu_name="unitree_imu" xyz="0. 0. 0." rpy="0. 0. 0."/>
-    <xacro:leg prefix="LF" mirror="1" mirror_dae="True" front_hind="1" front_hind_dae="True">
+    <xacro:leg prefix="LF" mesh_path="${mesh_path}" mirror="1" mirror_dae="True" front_hind="1" front_hind_dae="True">
         <origin rpy="0 0 0" xyz="${leg_offset_x} ${leg_offset_y} 0"/>
     </xacro:leg>
-    <xacro:leg prefix="LH" mirror="1" mirror_dae="True" front_hind="-1" front_hind_dae="False">
+    <xacro:leg prefix="LH" mesh_path="${mesh_path}" mirror="1" mirror_dae="True" front_hind="-1" front_hind_dae="False">
         <origin rpy="0 0 0" xyz="${-leg_offset_x} ${leg_offset_y} 0"/>
     </xacro:leg>
-    <xacro:leg prefix="RF" mirror="-1" mirror_dae="False" front_hind="1" front_hind_dae="True">
+    <xacro:leg prefix="RF" mesh_path="${mesh_path}" mirror="-1" mirror_dae="False" front_hind="1" front_hind_dae="True">
         <origin rpy="0 0 0" xyz="${leg_offset_x} ${-leg_offset_y} 0"/>
     </xacro:leg>
-    <xacro:leg prefix="RH" mirror="-1" mirror_dae="False" front_hind="-1" front_hind_dae="False">
+    <xacro:leg prefix="RH" mesh_path="${mesh_path}" mirror="-1" mirror_dae="False" front_hind="-1" front_hind_dae="False">
         <origin rpy="0 0 0" xyz="${-leg_offset_x} ${-leg_offset_y} 0"/>
     </xacro:leg>
